File: Hardware/Kicad/ESCV00/ESCV00.kicad_pcb (KiCad board)
At the start: 6 copper layers, 42 x 42 mm, 233 parts, among them J1 FC, Q101 BSZ018N04LS6, Q102 BSZ018N04LS6, Q103 BSZ018N04LS6, Q104 BSZ018N04LS6, Q105 BSZ018N04LS6, Q106 BSZ018N04LS6, Q201 BSZ018N04LS6, Q202 BSZ018N04LS6, Q203 BSZ018N04LS6, Q204 BSZ018N04LS6, Q205 BSZ018N04LS6, Q206 BSZ018N04LS6, Q301 BSZ018N04LS6, Q302 BSZ018N04LS6, Q303 BSZ018N04LS6, Q304 BSZ018N04LS6, Q305 BSZ018N04LS6, Q306 BSZ018N04LS6, Q401 BSZ018N04LS6, Q402 BSZ018N04LS6, Q403 BSZ018N04LS6, Q404 BSZ018N04LS6, Q405 BSZ018N04LS6, Q406 BSZ018N04LS6, U1 INA181A3IDBVR, U101 STM32F051K8U6, U102 DRV8300DRGER, U2 LMR16006YDDCR, U201 STM32F051K8U6, U202 DRV8300DRGER, U3 MCP1703AT-3302E_MB, U301 STM32F051K8U6, U302 DRV8300DRGER, U401 STM32F051K8U6, U402 DRV8300DRGER

Commit message: Boards follow the B0_EE part convention
- every real part uses the symbol/footprint/3D/datasheet named after its MPN in Kicad_Libs
- symbols keep only Reference, Value, Footprint, Datasheet, Description
  (MPN, Manufacturer, Verify, LCSC, Note fields removed; Verify notes moved to the Readme)
- schematic symbol caches rebuilt from the libraries, PCB footprints relinked with the
  same fields and 3D models as the library (connectivity unchanged)
- DNP and BOM attributes of the footprints match the symbols
- BOMs re-exported with kicad-cli
- ignore KiCad local history
Parts:
- D1: footprint eDiodes:D_SOD-123F -> eDiodes:PMEG6010CEH
- FB101, FB201, FB301, FB401: value 120R@100MHz -> BLM15PX121SN1D; footprint eChoke:L_0402_1005Metric -> eFerrite:BLM15PX121SN1D
- J1: value FC -> SM08B-SRSS-TB; footprint eConnector:JST_SH_SM08B-SRSS-TB_1x08-1MP_P1.00mm_Horizontal -> eConnector:SM08B-SRSS-TB
- L1: value 10uH SWPA3012S-100MT -> SWPA3012S100MT; footprint eCoil:L_Sunlord_SWPA3012S -> eCoil:SWPA3012S100MT
- Q101, Q102, Q103, Q104, Q105, Q106, Q201, Q202, Q203, Q204, Q205, Q206, Q301, Q302, Q303, Q304, Q305, Q306, Q401, Q402, Q403, Q404, Q405, Q406: value BSZ018N04LS6 -> BSZ018N04LS6ATMA1; footprint eTransistor:PQFN-8_3.3x3.3mm_P0.65mm_PowerFET -> eTransistor:BSZ018N04LS6ATMA1
- R1, R2, R3, R4: value 1mR 3W -> WSLP2512R0010FEA; footprint eResistor:R_2512_6332Metric -> eResistor:WSLP2512R0010FEA
- U1: footprint eAmplifier:SOT-23-6 -> eAmplifier:INA181A3IDBVR
- U101, U201, U301, U401: footprint eMCU:QFN-32-1EP_5x5mm_P0.5mm_EP3.45x3.45mm -> eMCU:STM32F051K8U6
- U102, U202, U302, U402: footprint eInterface:VQFN-24-1EP_4x4mm_P0.5mm_EP2.45x2.45mm -> eInterface:DRV8300DRGER
- U2: footprint eConverterDCDC:SOT-23-6 -> eConverterDCDC:LMR16006YDDCR
- U3: footprint eLinearReg:SOT-89-3 -> eLinearReg:MCP1703AT-3302E_MB
