File: Hardware/Kicad/FCV00/FCV00.kicad_pcb (KiCad board)
At the start: 4 copper layers, 36 x 36 mm, 139 parts, among them J1 USB_C_GCT_USB4105-GF-A, J2 ESC, J3 RX, J4 VTX, J5 CAM, J6 GPS, J7 AUX, Q1 2N7002, SW1 BOOT, U1 TPS54360BDDAR, U2 TPS54360BDDAR, U3 AP2112K-3.3TRG1, U4 AP2112K-3.3TRG1, U5 STM32F405RGT6, U6 ICM-42688-P, U7 LPS22DF, U8 W25Q128JVSIQ, U9 AT7456E, Y1 8MHz 12pF, Y2 27MHz 12pF

Commit message: Boards follow the B0_EE part convention
- every real part uses the symbol/footprint/3D/datasheet named after its MPN in Kicad_Libs
- symbols keep only Reference, Value, Footprint, Datasheet, Description
  (MPN, Manufacturer, Verify, LCSC, Note fields removed; Verify notes moved to the Readme)
- schematic symbol caches rebuilt from the libraries, PCB footprints relinked with the
  same fields and 3D models as the library (connectivity unchanged)
- DNP and BOM attributes of the footprints match the symbols
- BOMs re-exported with kicad-cli
- ignore KiCad local history
Parts:
- D1: footprint eDiodes:D_SMA -> eDiodes:SMAJ28A
- D2, D3: value PMEG6045ETP -> PMEG6045ETPX; footprint eDiodes:D_SOD-128 -> eDiodes:PMEG6045ETPX
- D4: footprint eDiodes:D_SOD-123F -> eDiodes:PMEG3020EH
- D5: value RED -> KT-0603R; footprint eLED:LED_0603_1608Metric -> eLED:KT-0603R
- D8: footprint eDiodes:SOT-23-6 -> eDiodes:USBLC6-2SC6
- D9: footprint eDiodes:D_SOD-123 -> eDiodes:1N4148W
- FB1: value 600R@100MHz -> BLM15AG601SN1D; footprint eChoke:L_0402_1005Metric -> eFerrite:BLM15AG601SN1D
- FB2: value 600R@100MHz -> BLM18AG601SN1D; footprint eChoke:L_0603_1608Metric -> eFerrite:BLM18AG601SN1D
- J1: value USB_C_GCT_USB4105-GF-A -> USB4105-GF-A; footprint eConnector:USB_C_Receptacle_GCT_USB4105-xx-A_16P_TopMnt_Horizontal -> eConnector:USB4105-GF-A
- J2: value ESC -> SM08B-SRSS-TB; footprint eConnector:JST_SH_SM08B-SRSS-TB_1x08-1MP_P1.00mm_Horizontal -> eConnector:SM08B-SRSS-TB
- J3: value RX -> SM04B-SRSS-TB; footprint eConnector:JST_SH_SM04B-SRSS-TB_1x04-1MP_P1.00mm_Horizontal -> eConnector:SM04B-SRSS-TB
- J4: value VTX -> SM06B-SRSS-TB; footprint eConnector:JST_SH_SM06B-SRSS-TB_1x06-1MP_P1.00mm_Horizontal -> eConnector:SM06B-SRSS-TB
- J5: value CAM -> SM03B-SRSS-TB; footprint eConnector:JST_SH_SM03B-SRSS-TB_1x03-1MP_P1.00mm_Horizontal -> eConnector:SM03B-SRSS-TB
- J6: value GPS -> SM06B-SRSS-TB; footprint eConnector:JST_SH_SM06B-SRSS-TB_1x06-1MP_P1.00mm_Horizontal -> eConnector:SM06B-SRSS-TB
- J7: value AUX -> SM06B-SRSS-TB; footprint eConnector:JST_SH_SM06B-SRSS-TB_1x06-1MP_P1.00mm_Horizontal -> eConnector:SM06B-SRSS-TB
- L1: value 6.8uH SRP5030T-6R8M -> SRP5030T-6R8M; footprint eCoil:L_Bourns_SRP5030T -> eCoil:SRP5030T-6R8M
- L2: value 10uH SRP5030T-100M -> SRP5030T-100M; footprint eCoil:L_Bourns_SRP5030T -> eCoil:SRP5030T-100M
- Q1: footprint eTransistor:SOT-23 -> eTransistor:2N7002
- SW1: value BOOT -> B3U-1000P; footprint eSwitch:SW_SPST_B3U-1000P -> eSwitch:B3U-1000P
- U1, U2: footprint eConverterDCDC:TI_SO-PowerPAD-8_ThermalVias -> eConverterDCDC:TPS54360BDDAR
- U3, U4: footprint eLinearReg:SOT-23-5 -> eLinearReg:AP2112K-3.3TRG1
- U5: footprint eMCU:LQFP-64_10x10mm_P0.5mm -> eMCU:STM32F405RGT6
- U6: footprint eSensor:Bosch_LGA-14_3x2.5mm_P0.5mm -> eSensor:ICM-42688-P
- U7: value LPS22DF -> LPS22DFTR; footprint eSensor:ST_HLGA-10_2x2mm_P0.5mm_LayoutBorder3x2y -> eSensor:LPS22DFTR
- U8: footprint eMemory:SOIC-8_5.23x5.23mm_P1.27mm -> eMemory:W25Q128JVSIQ
- U9: footprint eDisplay:HTSSOP-28-1EP_4.4x9.7mm_P0.65mm_EP2.85x5.4mm -> eDisplay:AT7456E
- Y1: value 8MHz 12pF -> X322508MLB4SI; footprint eCrystal:Crystal_SMD_3225-4Pin_3.2x2.5mm -> eCrystal:X322508MLB4SI
- Y2: value 27MHz 12pF -> X322527MOB4SI; footprint eCrystal:Crystal_SMD_3225-4Pin_3.2x2.5mm -> eCrystal:X322527MOB4SI
