File: Hardware/Kicad/FCV00/FCV00.kicad_sch (KiCad schematic)
At the start: 0 parts

Commit message: prima versione pcb
Other:
- added sheet Connectors (connectors.kicad_sch)
- added sheet MCU (mcu.kicad_sch)
- added sheet OSD (osd.kicad_sch)
- added sheet Power (power.kicad_sch)
- added sheet Sensors (sensors.kicad_sch)
- note added: "FCV00 - FLIGHT CONTROLLER MCU pin map (STM32F405RGT6) SPI1 PA5/PA6/PA7 CS PA4 INT PC4 CLKIN PB0 -> ICM-42688-P (gyro) SPI2 PB13/PB14/PB15 CS PB12 -> AT7456E (OSD) SPI3 PB3/PB4/PB5 CS PA15 -> W25Q128 (blackbox) I2C1 PB8/PB9 -> LPS22DF baro + GPS compass USART1 PB6/PB7 -> ELRS RX USART2 PA2/PA3 -> VTX (MSP/SmartAudio) USART3 PB10/PB11 -> GPS UART4 PA0/PA1 -> AUX UART5 PC12 (AUX TX) / PD2 (ESC telem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"
- company: (none) -> Drone project
- title: (none) -> Flight Controller - Overview
Changed lines of the file:
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@@
-(kicad_sch
-	(version 20250114)
-	(generator "eeschema")
-	(generator_version "9.0")
-	(paper "A4")
-	(sheet_instances
-		(path "/"
-			(page "1")
-		)
-	)
-	(embedded_fonts no)
+(kicad_sch (version 20230121) (generator eeschema)
+  (paper "A3")
+  (title_block
+    (title "Flight Controller - Overview")
+    (date "2026-10-08")
+    (rev "V00")
+    (company "Drone project")
+    (comment 1 "STM32F405RGT6 / ICM-42688-P / LPS22DF / AT7456E / W25Q128JV")
+    (comment 2 "Input 2S-6S (VBAT max 25.2V). 5V 3A + 10V 2A bucks, 2x 3.3V LDO")
+    (comment 3 "30.5x30.5 mm pattern, 4-layer 1.6mm")
+  )
+  (sheet (at 25.4 50.8) (size 40.64 15.24) (fields_autoplaced)
+    (stroke (width 0.1524) (type solid))
+    (fill (color 0 0 0 0.0000))
+    (property "Sheetname" "Power" (at 25.4 50.1 0)
+      (effects (font (size 1.27 1.27)) (justify left bottom))
+    )
+    (property "Sheetfile" "power.kicad_sch" (at 25.4 66.64 0)
+      (effects (font (size 1.27 1.27)) (justify left top))
+    )
+    (instances
+      (project "FCV00"
+        (path "/68a871cc-4819-5cae-bfd4-26989a952d6f" (page "2"))
+      )
+    )
+  )
+  (sheet (at 25.4 78.74) (size 40.64 15.24) (fields_autoplaced)
+    (stroke (width 0.1524) (type solid))
+    (fill (color 0 0 0 0.0000))
+    (property "Sheetname" "MCU" (at 25.4 78.04 0)
+      (effects (font (size 1.27 1.27)) (justify left bottom))
+    )
+    (property "Sheetfile" "mcu.kicad_sch" (at 25.4 94.58 0)
+      (effects (font (size 1.27 1.27)) (justify left top))
+    )
+    (instances
+      (project "FCV00"
+        (path "/68a871cc-4819-5cae-bfd4-26989a952d6f" (page "3"))
+      )
+    )
+  )
+  (sheet (at 25.4 106.68) (size 40.64 15.24) (fields_autoplaced)
+    (stroke (width 0.1524) (type solid))
+    (fill (color 0 0 0 0.0000))
+    (property "Sheetname" "Sensors" (at 25.4 105.98 0)
+      (effects (font (size 1.27 1.27)) (justify left bottom))
+    )
+    (property "Sheetfile" "sensors.kicad_sch" (at 25.4 122.52 0)
+      (effects (font (size 1.27 1.27)) (justify left top))
+    )
+    (instances
+      (project "FCV00"
+        (path "/68a871cc-4819-5cae-bfd4-26989a952d6f" (page "4"))
+      )
+    )
+  )
+  (sheet (at 25.4 134.62) (size 40.64 15.24) (fields_autoplaced)
+    (stroke (width 0.1524) (type solid))
+    (fill (color 0 0 0 0.0000))
+    (property "Sheetname" "OSD" (at 25.4 133.92 0)
+      (effects (font (size 1.27 1.27)) (justify left bottom))
+    )
+    (property "Sheetfile" "osd.kicad_sch" (at 25.4 150.46 0)
+      (effects (font (size 1.27 1.27)) (justify left top))
+    )
+    (instances
+      (project "FCV00"
+        (path "/68a871cc-4819-5cae-bfd4-26989a952d6f" (page "5"))
+      )
+    )
+  )
+  (sheet (at 25.4 162.56) (size 40.64 15.24) (fields_autoplaced)
+    (stroke (width 0.1524) (type solid))
+    (fill (color 0 0 0 0.0000))
+    (property "Sheetname" "Connectors" (at 25.4 161.86 0)
+      (effects (font (size 1.27 1.27)) (justify left bottom))
+    )
+    (property "Sheetfile" "connectors.kicad_sch" (at 25.4 178.4 0)
+      (effects (font (size 1.27 1.27)) (justify left top))
+    )
+    (instances
+      (project "FCV00"
+        (path "/68a871cc-4819-5cae-bfd4-26989a952d6f" (page "6"))
+      )
+    )
+  )
+  (text "FCV00 - FLIGHT CONTROLLER\nMCU pin map (STM32F405RGT6)\n  SPI1 PA5/PA6/PA7  CS PA4  INT PC4  CLKIN PB0 -> ICM-42688-P (gyro)\n  SPI2 PB13/PB14/PB15  CS PB12        -> AT7456E (OSD)\n  SPI3 PB3/PB4/PB5  CS PA15           -> W25Q128 (blackbox)\n  I2C1 PB8/PB9                        -> LPS22DF baro + GPS compass\n  USART1 PB6/PB7 -> ELRS RX     USART2 PA2/PA3 -> VTX (MSP/SmartAudio)\n  USART3 PB10/PB11 -> GPS       UART4 PA0/PA1 -> AUX\n  UART5 PC12 (AUX TX) / PD2 (ESC telemetry RX)\n  MOTOR1..4 PC6..PC9 = TIM8 CH1..CH4 (DShot / bidir DShot)\n  LED strip PA8 (TIM1 CH1)   Buzzer PC5   LEDs PC14/PC15\n  ADC: VBAT PC2 (x11 divider), CURRENT PC1, USB VBUS detect PA9\n" (at 180 20 0)
+    (effects (font (size 1.5 1.5)) (justify left top))
+  )
+  (sheet_instances
+    (path "/" (page "1"))
+  )
 )
