File: Hardware/Kicad/RXV00/RXV00.kicad_pcb (KiCad board)
At the start: 4 copper layers, 22 x 14 mm, 49 parts, among them J1 FC, J2 U.FL, SW1 BOOT, U1 AP2112K-3.3TRG1, U2 ESP32-C3FH4, U3 SX1281IMLTRT, Y1 40MHz 10pF, Y2 52MHz 8pF

Commit message: Boards follow the B0_EE part convention
- every real part uses the symbol/footprint/3D/datasheet named after its MPN in Kicad_Libs
- symbols keep only Reference, Value, Footprint, Datasheet, Description
  (MPN, Manufacturer, Verify, LCSC, Note fields removed; Verify notes moved to the Readme)
- schematic symbol caches rebuilt from the libraries, PCB footprints relinked with the
  same fields and 3D models as the library (connectivity unchanged)
- DNP and BOM attributes of the footprints match the symbols
- BOMs re-exported with kicad-cli
- ignore KiCad local history
Parts:
- AE1: value 2450AT18A100 -> 2450AT18A100E; footprint eAntenna:Johanson_2450AT18x100 -> eAntenna:2450AT18A100E
- FB1: value 120R@100MHz -> BLM15PX121SN1D; footprint eChoke:L_0402_1005Metric -> eFerrite:BLM15PX121SN1D
- J1: value FC -> SM04B-SRSS-TB; footprint eConnector:JST_SH_SM04B-SRSS-TB_1x04-1MP_P1.00mm_Horizontal -> eConnector:SM04B-SRSS-TB
- J2: value U.FL -> U.FL-R-SMT-1; footprint eConnector:U.FL_Hirose_U.FL-R-SMT-1_Vertical -> eConnector:U.FL-R-SMT-1
- L2: value 15uH -> LQM21PN150MC0; footprint eCoil:L_0805_2012Metric -> eCoil:LQM21PN150MC0
- L3: value 47nH (tune) -> LQW15AN47NJ00D; footprint eCoil:L_0402_1005Metric -> eCoil:LQW15AN47NJ00D
- L4: value 4.7nH -> LQP15MN4N7B02D; footprint eCoil:L_0402_1005Metric -> eCoil:LQP15MN4N7B02D
- SW1: value BOOT -> B3U-1000P; footprint eSwitch:SW_SPST_B3U-1000P -> eSwitch:B3U-1000P
- U1: footprint eLinearReg:SOT-23-5 -> eLinearReg:AP2112K-3.3TRG1
- U2: footprint eMCU:QFN-32-1EP_5x5mm_P0.5mm_EP3.7x3.7mm -> eMCU:ESP32-C3FH4
- U3: footprint eRFModule:QFN-24-1EP_4x4mm_P0.5mm_EP2.6x2.6mm -> eRFModule:SX1281IMLTRT
- Y1: value 40MHz 10pF -> X201640MLB4SI; footprint eCrystal:Crystal_SMD_2016-4Pin_2.0x1.6mm -> eCrystal:X201640MLB4SI
- Y2: value 52MHz 8pF -> X201652MOB4SI; footprint eCrystal:Crystal_SMD_2016-4Pin_2.0x1.6mm -> eCrystal:X201652MOB4SI
