File: Hardware/Kicad/VTXV00/VTXV00.kicad_pcb (KiCad board)
At the start: 4 copper layers, 27 x 27 mm, 85 parts, among them J1 FC, J2 U.FL, Q1 MMBT3904, SW1 BAND/CH, U1 AP2112K-3.3TRG1, U2 STM32F031G6U6, U3 RTC6705, U4 RFPA5542, Y1 8MHz 12pF

Commit message: Boards follow the B0_EE part convention
- every real part uses the symbol/footprint/3D/datasheet named after its MPN in Kicad_Libs
- symbols keep only Reference, Value, Footprint, Datasheet, Description
  (MPN, Manufacturer, Verify, LCSC, Note fields removed; Verify notes moved to the Readme)
- schematic symbol caches rebuilt from the libraries, PCB footprints relinked with the
  same fields and 3D models as the library (connectivity unchanged)
- DNP and BOM attributes of the footprints match the symbols
- BOMs re-exported with kicad-cli
- ignore KiCad local history
Parts:
- FB1: value 120R 3A -> BLM18KG121TN1D; footprint eChoke:L_0603_1608Metric -> eFerrite:BLM18KG121TN1D
- FB2: value 120R@100MHz -> BLM18PG121SN1D; footprint eChoke:L_0603_1608Metric -> eFerrite:BLM18PG121SN1D
- J1: value FC -> SM06B-SRSS-TB; footprint eConnector:JST_SH_SM06B-SRSS-TB_1x06-1MP_P1.00mm_Horizontal -> eConnector:SM06B-SRSS-TB
- J2: value U.FL -> U.FL-R-SMT-1; footprint eConnector:U.FL_Hirose_U.FL-R-SMT-1_Vertical -> eConnector:U.FL-R-SMT-1
- Q1: value MMBT3904 -> MMBT3904LT1G; footprint eTransistor:SOT-23 -> eTransistor:MMBT3904LT1G
- SW1: value BAND/CH -> B3U-1000P; footprint eSwitch:SW_SPST_B3U-1000P -> eSwitch:B3U-1000P
- U1: footprint eLinearReg:SOT-23-5 -> eLinearReg:AP2112K-3.3TRG1
- U2: footprint eMCU:QFN-28_4x4mm_P0.5mm -> eMCU:STM32F031G6U6
- U3: footprint eRFModule:QFN-40-1EP_6x6mm_P0.5mm_EP4.6x4.6mm -> eRFModule:RTC6705
- U4: value RFPA5542 -> RFPA5542TR13; footprint eAmplifier:QFN-20-1EP_4x4mm_P0.5mm_EP2.5x2.5mm -> eAmplifier:RFPA5542TR13
- Y1: value 8MHz 12pF -> X322508MLB4SI; footprint eCrystal:Crystal_SMD_3225-4Pin_3.2x2.5mm -> eCrystal:X322508MLB4SI
Changed lines of the file:
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@@
 		)
 	)
-	(footprint "eTransistor:SOT-23"
+	(footprint "eTransistor:MMBT3904LT1G"
 		(layer "F.Cu")
 		(at 93.945 60.86)
@@
 			)
 		)
-		(property "Value" "MMBT3904"
+		(property "Value" "MMBT3904LT1G"
 			(at 0 2.4 0)
 			(layer "F.Fab")
@@
 			)
 		)
-		(property "Datasheet" ""
+		(property "Datasheet" "${KIPRJMOD}/../KiCad_Libs/eTransistor/datasheet/MMBT3904LT1G.pdf"
 			(at 0 0 0)
 			(layer "F.Fab")
@@
 			)
 		)
-		(property "Description" ""
+		(property "Description" "NPN transistor, 40 V, 200 mA, SOT-23"
 			(at 0 0 0)
 			(layer "F.Fab")
@@
 		)
 		(embedded_fonts no)
-		(model "${KIPRJMOD}/../KiCad_Libs/eTransistor/eTransistor.3dshapes/SOT-23.step"
+		(model "${KIPRJMOD}/../KiCad_Libs/eTransistor/eTransistor.3dshapes/MMBT3904LT1G.step"
 			(offset
 				(xyz 0 0 0)
@@
 			)
 		)
-		(attr smd exclude_from_bom)
+		(attr smd dnp)
 		(duplicate_pad_numbers_are_jumpers no)
 		(fp_line
@@
 			)
 		)
-		(attr smd exclude_from_bom)
+		(attr smd dnp)
 		(duplicate_pad_numbers_are_jumpers no)
 		(fp_line
@@
 		)
 	)
-	(footprint "eRFModule:QFN-40-1EP_6x6mm_P0.5mm_EP4.6x4.6mm"
+	(footprint "eRFModule:RTC6705"
 		(layer "F.Cu")
 		(at 103.645 73.21)
@@
 			)
 		)
-		(property "Datasheet" ""
+		(property "Datasheet" "${KIPRJMOD}/../KiCad_Libs/eRFModule/datasheet/RTC6705.pdf"
 			(at 0 0 0)
 			(layer "F.Fab")
@@
 			)
 		)
-		(property "Description" ""
+		(property "Description" "5.8 GHz FM video transmitter with PLL, QFN-40"
 			(at 0 0 0)
 			(layer "F.Fab")
@@
 		)
 		(embedded_fonts no)
-		(model "${KIPRJMOD}/../KiCad_Libs/eRFModule/eRFModule.3dshapes/QFN-40-1EP_6x6mm_P0.5mm_EP4.6x4.6mm.step"
+		(model "${KIPRJMOD}/../KiCad_Libs/eRFModule/eRFModule.3dshapes/RTC6705.step"
 			(offset
 				(xyz 0 0 0)
@@
 		(embedded_fonts no)
 	)
-	(footprint "eChoke:L_0603_1608Metric"
+	(footprint "eFerrite:BLM18KG121TN1D"
 		(layer "F.Cu")
 		(at 111.675 47.755)
@@
 			)
 		)
-		(property "Value" "120R 3A"
+		(property "Value" "BLM18KG121TN1D"
 			(at 0 1.43 0)
 			(layer "F.Fab")
@@
 			)
 		)
-		(property "Datasheet" ""
+		(property "Datasheet" "${KIPRJMOD}/../KiCad_Libs/eFerrite/datasheet/BLM18KG121TN1D.pdf"
 			(at 0 0 0)
 			(layer "F.Fab")
@@
 			)
 		)
-		(property "Description" ""
+		(property "Description" "Ferrite bead, 120 Ohm @ 100 MHz, 3 A, 0603"
 			(at 0 0 0)
 			(layer "F.Fab")
@@
 		)
 		(embedded_fonts no)
-		(model "${KIPRJMOD}/../KiCad_Libs/eChoke/eChoke.3dshapes/L_0603_1608Metric.step"
+		(model "${KIPRJMOD}/../KiCad_Libs/eFerrite/eFerrite.3dshapes/BLM18KG121TN1D.step"
 			(offset
 				(xyz 0 0 0)
@@
 		)
 	)
-	(footprint "eCrystal:Crystal_SMD_3225-4Pin_3.2x2.5mm"
+	(footprint "eCrystal:X322508MLB4SI"
 		(layer "F.Cu")
 		(at 139.094999 71.31)
@@
 			)
 		)
-		(property "Value" "8MHz 12pF"
+		(property "Value" "X322508MLB4SI"
 			(at 0 2.45 0)
 			(layer "F.Fab")
@@
 			)
 		)
-		(property "Datasheet" ""
+		(property "Datasheet" "${KIPRJMOD}/../KiCad_Libs/eCrystal/datasheet/X322508MLB4SI.pdf"
 			(at 0 0 0)
 			(layer "F.Fab")
@@
 			)
 		)
-		(property "Description" ""
+		(property "Description" "Crystal, 8 MHz, 12 pF, SMD3225-4P"
 			(at 0 0 0)
 			(layer "F.Fab")
@@
 		)
 		(embedded_fonts no)
-		(model "${KIPRJMOD}/../KiCad_Libs/eCrystal/eCrystal.3dshapes/Crystal_SMD_3225-4Pin_3.2x2.5mm.step"
+		(model "${KIPRJMOD}/../KiCad_Libs/eCrystal/eCrystal.3dshapes/X322508MLB4SI.step"
 			(offset
 				(xyz 0 0 0)
@@
 		)
 	)
-	(footprint "eConnector:U.FL_Hirose_U.FL-R-SMT-1_Vertical"
+	(footprint "eConnector:U.FL-R-SMT-1"
 		(layer "F.Cu")
 		(at 129.074999 82.87)
@@
 			)
 		)
-		(property "Value" "U.FL"
+		(property "Value" "U.FL-R-SMT-1"
 			(at 0.475 3.2 0)
 			(layer "F.Fab")
@@
 			)
 		)
-		(property "Datasheet" ""
+		(property "Datasheet" "${KIPRJMOD}/../KiCad_Libs/eConnector/datasheet/U.FL-R-SMT-1.pdf"
 			(at 0 0 0)
 			(layer "F.Fab")
@@
 			)
 		)
-		(property "Description" ""
+		(property "Description" "U.FL coaxial receptacle, 50 Ohm, 6 GHz, SMD"
 			(at 0 0 0)
 			(layer "F.Fab")
@@
 		)
 		(embedded_fonts no)
-		(model "${KIPRJMOD}/../KiCad_Libs/eConnector/eConnector.3dshapes/U.FL_Hirose_U.FL-R-SMT-1_Vertical.step"
+		(model "${KIPRJMOD}/../KiCad_Libs/eConnector/eConnector.3dshapes/U.FL-R-SMT-1.step"
 			(offset
 				(xyz 0 0 0)
@@
 			)
 		)
-		(attr smd exclude_from_bom)
+		(attr smd dnp)
 		(duplicate_pad_numbers_are_jumpers no)
 		(fp_line
@@
 		)
 	)
-	(footprint "eLinearReg:SOT-23-5"
+	(footprint "eLinearReg:AP2112K-3.3TRG1"
 		(layer "F.Cu")
 		(at 120.705 48.9)
@@
 			)
 		)
-		(property "Datasheet" ""
+		(property "Datasheet" "${KIPRJMOD}/../KiCad_Libs/eLinearReg/datasheet/AP2112K-3.3TRG1.pdf"
 			(at 0 0 0)
 			(layer "F.Fab")
@@
 			)
 		)
-		(property "Description" ""
+		(property "Description" "LDO regulator, 3.3 V, 600 mA, with enable, SOT-23-5"
 			(at 0 0 0)
 			(layer "F.Fab")
@@
 		)
 		(embedded_fonts no)
-		(model "${KIPRJMOD}/../KiCad_Libs/eLinearReg/eLinearReg.3dshapes/SOT-23-5.step"
+		(model "${KIPRJMOD}/../KiCad_Libs/eLinearReg/eLinearReg.3dshapes/AP2112K-3.3TRG1.step"
 			(offset
 				(xyz 0 0 0)
@@
 			)
 		)
-		(attr smd exclude_from_bom)
+		(attr smd dnp)
 		(duplicate_pad_numbers_are_jumpers no)
 		(fp_line
@@
 		)
 	)
-	(footprint "eSwitch:SW_SPST_B3U-1000P"
+	(footprint "eSwitch:B3U-1000P"
 		(layer "F.Cu")
 		(at 124.034999 56.285)
@@
 			)
 		)
-		(property "Value" "BAND/CH"
+		(property "Value" "B3U-1000P"
 			(at 0 2.5 0)
 			(layer "F.Fab")
@@
 			)
 		)
-		(property "Datasheet" ""
+		(property "Datasheet" "${KIPRJMOD}/../KiCad_Libs/eSwitch/datasheet/B3U-1000P.pdf"
 			(at 0 0 0)
 			(layer "F.Fab")
@@
 			)
 		)
-		(property "Description" ""
+		(property "Description" "Tactile switch, SPST-NO, 3.0x2.5 mm, SMD"
 			(at 0 0 0)
 			(layer "F.Fab")
@@
 		)
 		(embedded_fonts no)
-		(model "${KIPRJMOD}/../KiCad_Libs/eSwitch/eSwitch.3dshapes/SW_SPST_B3U-1000P.step"
+		(model "${KIPRJMOD}/../KiCad_Libs/eSwitch/eSwitch.3dshapes/B3U-1000P.step"
 			(offset
 				(xyz 0 0 0)
@@
 			)
 		)
-		(attr smd exclude_from_bom)
+		(attr smd dnp)
 		(duplicate_pad_numbers_are_jumpers no)
 		(fp_line
@@
 			)
 		)
-		(attr smd exclude_from_bom)
+		(attr smd dnp)
 		(duplicate_pad_numbers_are_jumpers no)
 		(fp_line
@@
 		)
 	)
-	(footprint "eAmplifier:QFN-20-1EP_4x4mm_P0.5mm_EP2.5x2.5mm"
+	(footprint "eAmplifier:RFPA5542TR13"
 		(layer "F.Cu")
 		(at 94.625 82.97)
@@
 			)
 		)
-		(property "Value" "RFPA5542"
+		(property "Value" "RFPA5542TR13"
 			(at 0 3.3 0)
 			(layer "F.Fab")
@@
 			)
 		)
-		(property "Datasheet" ""
+		(property "Datasheet" "${KIPRJMOD}/../KiCad_Libs/eAmplifier/datasheet/RFPA5542TR13.pdf"
 			(at 0 0 0)
 			(layer "F.Fab")
@@
 			)
 		)
-		(property "Description" ""
+		(property "Description" "5 GHz WLAN power amplifier, 4.9 to 5.9 GHz, QFN-20"
 			(at 0 0 0)
 			(layer "F.Fab")
@@
 		)
 		(embedded_fonts no)
-		(model "${KIPRJMOD}/../KiCad_Libs/eAmplifier/eAmplifier.3dshapes/QFN-20-1EP_4x4mm_P0.5mm_EP2.5x2.5mm.step"
+		(model "${KIPRJMOD}/../KiCad_Libs/eAmplifier/eAmplifier.3dshapes/RFPA5542TR13.step"
 			(offset
 				(xyz 0 0 0)
@@
 		)
 	)
-	(footprint "eMCU:QFN-28_4x4mm_P0.5mm"
+	(footprint "eMCU:STM32F031G6U6"
 		(layer "F.Cu")
 		(at 133.315 49.655)
@@
 			)
 		)
-		(property "Datasheet" ""
+		(property "Datasheet" "${KIPRJMOD}/../KiCad_Libs/eMCU/datasheet/STM32F031G6U6.pdf"
 			(at 0 0 0)
 			(layer "F.Fab")
@@
 			)
 		)
-		(property "Description" ""
+		(property "Description" "ARM Cortex-M0 MCU, 32 KB flash, 4 KB RAM, 48 MHz, UFQFPN-28"
 			(at 0 0 0)
 			(layer "F.Fab")
@@
 		)
 		(embedded_fonts no)
-		(model "${KIPRJMOD}/../KiCad_Libs/eMCU/eMCU.3dshapes/QFN-28_4x4mm_P0.5mm.step"
+		(model "${KIPRJMOD}/../KiCad_Libs/eMCU/eMCU.3dshapes/STM32F031G6U6.step"
 			(offset
 				(xyz 0 0 0)
@@
 		)
 	)
-	(footprint "eConnector:JST_SH_SM06B-SRSS-TB_1x06-1MP_P1.00mm_Horizontal"
+	(footprint "eConnector:SM06B-SRSS-TB"
 		(layer "F.Cu")
 		(at 96.925 50.305)
@@
 			)
 		)
-		(property "Value" "FC"
+		(property "Value" "SM06B-SRSS-TB"
 			(at 0 3.98 0)
 			(layer "F.Fab")
@@
 			)
 		)
-		(property "Datasheet" ""
+		(property "Datasheet" "${KIPRJMOD}/../KiCad_Libs/eConnector/datasheet/SM06B-SRSS-TB.pdf"
 			(at 0 0 0)
 			(layer "F.Fab")
@@
 			)
 		)
-		(property "Description" ""
+		(property "Description" "JST SH connector header, 6 pin, 1.0 mm pitch, side entry, SMD"
 			(at 0 0 0)
 			(layer "F.Fab")
@@
 		)
 		(embedded_fonts no)
-		(model "${KIPRJMOD}/../KiCad_Libs/eConnector/eConnector.3dshapes/JST_SH_SM06B-SRSS-TB_1x06-1MP_P1.00mm_Horizontal.step"
+		(model "${KIPRJMOD}/../KiCad_Libs/eConnector/eConnector.3dshapes/SM06B-SRSS-TB.step"
 			(offset
 				(xyz 0 0 0)
@@
 		)
 	)
-	(footprint "eChoke:L_0603_1608Metric"
+	(footprint "eFerrite:BLM18PG121SN1D"
 		(layer "F.Cu")
 		(at 93.505 70.34)
@@
 			)
 		)
-		(property "Value" "120R@100MHz"
+		(property "Value" "BLM18PG121SN1D"
 			(at 0 1.43 0)
 			(layer "F.Fab")
@@
 			)
 		)
-		(property "Datasheet" ""
+		(property "Datasheet" "${KIPRJMOD}/../KiCad_Libs/eFerrite/datasheet/BLM18PG121SN1D.pdf"
 			(at 0 0 0)
 			(layer "F.Fab")
@@
 			)
 		)
-		(property "Description" ""
+		(property "Description" "Ferrite bead, 120 Ohm @ 100 MHz, 2 A, 0603"
 			(at 0 0 0)
 			(layer "F.Fab")
@@
 		)
 		(embedded_fonts no)
-		(model "${KIPRJMOD}/../KiCad_Libs/eChoke/eChoke.3dshapes/L_0603_1608Metric.step"
+		(model "${KIPRJMOD}/../KiCad_Libs/eFerrite/eFerrite.3dshapes/BLM18PG121SN1D.step"
 			(offset
 				(xyz 0 0 0)
